Commit message: test branch commit 2DOF_robot_arm

File: 2dof_robot_arm_assembly_description/urdf/2dof_robot_arm_assembly.xacro (robot description, xacro)
@@ -15,5 +15,5 @@
       <mesh filename="package://2dof_robot_arm_assembly_description/meshes/base_link.stl" scale="0.001 0.001 0.001"/>
     </geometry>
-    <material name="_"/>
+    <material name="steel_satin"/>
   </visual>
   <collision>
@@ -35,5 +35,5 @@
       <mesh filename="package://2dof_robot_arm_assembly_description/meshes/link1_v3_1.stl" scale="0.001 0.001 0.001"/>
     </geometry>
-    <material name="_"/>
+    <material name="steel_satin"/>
   </visual>
   <collision>
@@ -55,5 +55,5 @@
       <mesh filename="package://2dof_robot_arm_assembly_description/meshes/link2_v1_1.stl" scale="0.001 0.001 0.001"/>
     </geometry>
-    <material name="_"/>
+    <material name="steel_satin"/>
   </visual>
   <collision>
@@ -75,5 +75,5 @@
       <mesh filename="package://2dof_robot_arm_assembly_description/meshes/end_effector_v2_1.stl" scale="0.001 0.001 0.001"/>
     </geometry>
-    <material name="_"/>
+    <material name="steel_satin"/>
   </visual>
   <collision>
@@ -84,5 +84,5 @@
   </collision>
 </link>
-<joint name="��]1" type="continuous">
+<joint name="Rev1" type="continuous">
   <origin xyz="0.0 0.0 0.04" rpy="0 0 0"/>
   <parent link="base_link"/>
@@ -90,5 +90,5 @@
   <axis xyz="0.0 0.0 1.0"/>
 </joint>
-<joint name="��]2" type="revolute">
+<joint name="Rev2" type="revolute">
   <origin xyz="0.0011 -0.009939 0.03" rpy="0 0 0"/>
   <parent link="link1_v3_1"/>
@@ -97,5 +97,5 @@
   <limit upper="1.22173" lower="-1.22173" effort="100" velocity="100"/>
 </joint>
-<joint name="��]3" type="revolute">
+<joint name="Rev3" type="revolute">
   <origin xyz="0.071318 0.022983 0.0679" rpy="0 0 0"/>
   <parent link="link2_v1_1"/>

File: 2dof_robot_arm_assembly_description/urdf/materials.xacro (robot description, xacro)
@@ -4,5 +4,5 @@
   <color rgba="0.700 0.700 0.700 1.000"/>
 </material>
-<material name="_">
+<material name="steel_satin">
   <color rgba="0.6274509803921569 0.6274509803921569 0.6274509803921569 1.0"/>
 </material>
